File: hardware/leddriver/LED_driverV1.sch (EAGLE design)
At the start: 45 parts, among them IC1 ATTINY24/44/84-SSU, IC3 78L05SMD, Q1 BC807-40SMD, Q2 BC817-40SMD, Q3 BC817-40SMD, Q4 BSS123, Q5 BSS123, Q6 BSS123, T1 IRLR3410, Y1 CRYSTAL.3.2X2.5MM

Commit message: Hardware fixes + probably fixed PCB layout
Parts:
- R10: value 47k -> 39k
- R12: value 3k3 -> 1k
- R13: value 1k -> 3k3
- R3: value 330 -> 10
- R4: value 20 -> 10
Changed lines of the file:
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@@
 <part name="Q3" library="transistor-npn" deviceset="BC817*" device="SMD" technology="-40"/>
 <part name="R2" library="rcl" deviceset="R-EU_" device="R0603" value="330"/>
-<part name="R3" library="rcl" deviceset="R-EU_" device="R0603" value="330"/>
-<part name="R4" library="rcl" deviceset="R-EU_" device="R0603" value="20"/>
+<part name="R3" library="rcl" deviceset="R-EU_" device="R0603" value="10"/>
+<part name="R4" library="rcl" deviceset="R-EU_" device="R0603" value="10"/>
 <part name="P+4" library="supply1" deviceset="+12V" device=""/>
 <part name="GND8" library="supply1" deviceset="GND" device=""/>
@@
 <part name="R8" library="rcl" deviceset="R-EU_" device="R0603" value="1k"/>
 <part name="R9" library="rcl" deviceset="R-EU_" device="R0603" value="1k"/>
-<part name="R10" library="rcl" deviceset="R-EU_" device="R0603" value="47k"/>
+<part name="R10" library="rcl" deviceset="R-EU_" device="R0603" value="39k"/>
 <part name="GND11" library="supply1" deviceset="GND" device=""/>
 <part name="IC3" library="linear" deviceset="78L*SMD" device="" technology="05"/>
@@
 <part name="12V" library="wirepad" deviceset="WIREPAD" device="SMD5-2,5"/>
 <part name="R14" library="rcl" deviceset="R-EU_" device="R0603" value="10k"/>
-<part name="R12" library="rcl" deviceset="R-EU_" device="R0603" value="3k3"/>
+<part name="R12" library="rcl" deviceset="R-EU_" device="R0603" value="1k"/>
 <part name="GND5" library="supply1" deviceset="GND" device=""/>
-<part name="R13" library="rcl" deviceset="R-EU_" device="R0603" value="1k"/>
+<part name="R13" library="rcl" deviceset="R-EU_" device="R0603" value="3k3"/>
 <part name="R15" library="ptc-ntc" deviceset="NTC640" device=""/>
 <part name="P+7" library="supply1" deviceset="+5V" device=""/>
