File: hardware/leddriver/LED_driverV1_1.brd (EAGLE design)
At the start: 50 x 50 mm, 45 parts, among them IC1 ATTINY24/44/84-SSU, IC3 78L05SMD, Q1 BC807-40SMD, Q2 BC817-40SMD, Q3 BC817-40SMD, Q4 BSS123, Q5 BSS123, Q6 BSS123, T1 IRLR3410, Y1 CRYSTAL.3.2X2.5MM

Commit message: Hardware fixes + probably fixed PCB layout
Parts:
- removed Q3: BC817-40SMD, transistor-npn:SOT23-BEC
- removed R14: 10k, rcl:R0603
- added C13, C6, C7: 100n, rcl:C0603K
- added R11: 1k, rcl:R0603
- R10: value 47k -> 39k
- R12: value 3k3 -> 1k
- R13: value 1k -> 3k3
- R2: value 330 -> 10k
- R3: value 330 -> 10
- R4: value 20 -> 10
- moved R2 13.3 mm to (19.1, 10.2), turned to 270 degrees
- moved R3 3.86 mm to (26.7, 8.57)
- moved R8 1.60 mm to (31.1, 11.3)
Connections:
- removed net N$8: Q3.B, R14.1, R3.1
- net +12V: no longer R14.2, R2.2
- net ADC_I: now also C6.2
- net ADC_U: now also C7.1
- net GND: now also C13.1, C6.1, C7.2, R11.1, R2.1; no longer Q3.E
- net MISO: now also R11.2
- net PP_IN: now also R2.2, R3.1; no longer Q3.C, R2.1
- net TEMP: now also C13.2
Routing:
- net +5V: track 76.4 -> 58.0 mm, vias 5 -> 4
- net MISO: track 15.9 -> 25.8 mm
- net N$8: track 8.30 -> 0.00 mm
- net +12V: track 45.8 -> 38.0 mm
- net PP_IN: track 23.3 -> 18.9 mm
- net PWM: track 15.1 -> 19.2 mm
- net GND: track 86.2 -> 89.6 mm, vias 82 -> 78
- net ADC_I: track 2.90 -> 5.83 mm
- net TEMP: track 3.68 -> 5.71 mm
- net SCK: track 60.5 -> 61.9 mm
- net ADC_U: track 10.0 -> 11.5 mm
- net MOSI: track 69.0 -> 69.7 mm
- net CH1: track 19.5 -> 20.0 mm
Other:
- board text added: "LED driver V1.1"
- board text removed: "LED driver V1"
